File: Schematics/logic_board.sch (KiCad schematic (older format))
At the start: 0 parts

Commit message: Tja
Parts:
- added A1: Arduino, Module:Arduino_Nano, symbol Solder-station-rescue:Arduino_Nano_v2.x-MCU_Module
- added C10, C11: 0,1uF, symbol Solder-station-rescue:C-Device
- added C12, C13: 0,1uF, symbol Solder-station-rescue:CP-Device
- added J11: To power board, symbol Solder-station-rescue:Conn_02x05_Counter_Clockwise-Connector_Generic
- added J12: mains_sw, symbol Solder-station-rescue:Conn_01x01_Female-Connector
- added J13: airgun_sw, symbol Solder-station-rescue:Conn_01x01_Female-Connector
- added J14: Airgun_temp, symbol Solder-station-rescue:Conn_01x02-Connector_Generic
- added J15: Iron_temp, symbol Solder-station-rescue:Conn_01x02-Connector_Generic
- added R12: 470R, symbol Solder-station-rescue:R-Device
- added R13: 82R, symbol Solder-station-rescue:R-Device
- added R14: 100R, symbol Solder-station-rescue:R-Device
- added R15: 10k, symbol Solder-station-rescue:R-Device
- added R16, R17: 6k8, symbol Solder-station-rescue:R-Device
- added R8, R9, R?: 1k, symbol Solder-station-rescue:R-Device
- added R?: 270, symbol Solder-station-rescue:R-Device
- added SW2: Rotary_Switch, symbol Solder-station-rescue:Rotary_Encoder_Switch-Device
- added SW_blue1: blue_sw, symbol Solder-station-rescue:SW_Push_LED-Switch
- added SW_orag1: orag_sw, symbol Solder-station-rescue:SW_Push_LED-Switch
- added U5: ULN2803A, symbol Solder-station-rescue:ULN2803A-Transistor_Array
- added U6: TL082, symbol Solder-station-rescue:TL072-Amplifier_Operational
- added U7: Chassis_temp, symbol Solder-station-rescue:AD_tmp_sens-DIV_custom
- added U8: SH1106, symbol Solder-station-rescue:SH1106-DIV_custom
Connections:
- new net: A1.10 (D7), U5.3 (I3)
- new net: A1.11 (D8), U5.4 (I4)
- new net: A1.12 (D9), U5.5 (I5)
- new net: A1.13 (D10), J11.2 (Pin_2)
- new net: A1.14 (D11), U5.7 (I7)
- new net: A1.15 (D12), U5.8 (I8)
- new net: A1.16 (D13), J12.1 (Pin_1)
- new net: A1.19 (A0), J13.1 (Pin_1)
- new net: A1.20 (A1), SW_blue1.1
- new net: A1.21 (A2), SW_orag1.1
- new net: A1.22 (A3), U7.1 (A0)
- new net: A1.23 (A4), U8.3 (SDA)
- new net: A1.24 (A5), U8.4 (SCL)
- new net: A1.25 (A6), R17.2, U6.7
- new net: A1.26 (A7), R16.2, U6.1
- new net: A1.5 (D2), C11.1, R8.2
- new net: A1.6 (D3), C10.1, R9.2
- new net: A1.7 (D4), SW2.S1
- new net: A1.8 (D5), U5.1 (I1)
- new net: A1.9 (D6), U5.2 (I2)
- new net: R8.1, SW2.A
- new net: R9.1, SW2.B
- new net: SW_blue1.3 (K), U5.12 (O7)
- new net: R?.2, SW_blue1.4 (A)
- new net: SW_orag1.3 (K), U5.11 (O8)
- new net: R?.2, SW_orag1.4 (A)
- new net: U7.3 (GND), U8.1 (GND)
- new net: R12.1, R16.1, U6.2 (-)
- new net: C13.1, J15.1 (Pin_1), R15.2, U6.3 (+)
- new net: C12.1, J14.1 (Pin_1), R14.2, U6.5 (+)
- new net: R13.1, R17.1, U6.6 (-)
- new net: J11.4 (Pin_4), U5.14 (O5)
- new net: J11.6 (Pin_6), U5.15 (O4)
- new net: J11.7 (Pin_7), U5.16 (O3)
- new net: J11.9 (Pin_9), U5.17 (O2)
- new net: J11.10 (Pin_10), U5.18 (O1)
- new net +5V: A1.30 (VIN), J11.1 (Pin_1), R14.1, R15.1, R?.1, R?.1, U6.8 (V+), U7.4 (VCC), U8.2 (VCC)
- new net GNDREF: A1.29 (GND), A1.4 (GND), C10.2, C11.2, C12.2, C13.2, J11.5 (Pin_5), J14.2 (Pin_2), J15.2 (Pin_2), R12.2, R13.2, SW2.C, SW2.S2, SW_blue1.2, SW_orag1.2, U5.9 (GND), U6.4 (V-)
