File: Schematics/power_board.sch (KiCad schematic (older format))
At the start: 41 parts

Commit message: Tja
Parts:
- C1, C2: renamed from C?; symbol Device:C -> Solder-station-rescue:C-Device
- C3, C4, C5, C6, C7, C8, C9: renamed from C?; symbol Device:CP -> Solder-station-rescue:CP-Device
- D1, D2: renamed from D?; symbol Device:D -> Solder-station-rescue:D-Device
- D3, D4: renamed from D?; symbol Device:D_Bridge_+-AA -> Solder-station-rescue:D_Bridge_+-AA-Device
- F1: renamed from F?; symbol Device:Fuse -> Solder-station-rescue:Fuse-Device
- J1, J10, J2, J3, J4, J6, J7, J8, J9: renamed from J?; symbol Connector_Generic:Conn_01x02 -> Solder-station-rescue:Conn_01x02-Connector_Generic
- J5: renamed from J?; symbol Connector_Generic:Conn_02x05_Counter_Clockwise -> Solder-station-rescue:Conn_02x05_Counter_Clockwise-Connector_Generic
- K1, K2: renamed from K?; symbol DIV_custom:G2R-2-SN -> Solder-station-rescue:G2R-2-SN-DIV_custom
- Q1: renamed from Q?; symbol Transistor_BJT:TIP122 -> Solder-station-rescue:TIP122-Transistor_BJT
- Q2, Q3: renamed from Q?; symbol Triac_Thyristor:BT136-600 -> Solder-station-rescue:BT136-600-Triac_Thyristor
- R1, R2, R3, R4, R5, R6, R7: renamed from R?; symbol Device:R -> Solder-station-rescue:R-Device
- SW1: renamed from SW?; symbol Switch:SW_DPDT_x2 -> Solder-station-rescue:SW_DPDT_x2-Switch
- U1: renamed from U?; symbol Regulator_Linear:L7824 -> Solder-station-rescue:L7824-Regulator_Linear
- U2: renamed from U?; symbol Regulator_Linear:L7805 -> Solder-station-rescue:L7805-Regulator_Linear
- U3, U4: renamed from U?; symbol Relay_SolidState:MOC3041M -> Solder-station-rescue:MOC3041M-Relay_SolidState
Connections:
- net at C1.2, D1.2 (A), J1.2 (Pin_2)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: now also C6.1
- net at J5.2 (Pin_2), R1.2: no longer C6.1
Other:
- moved on the sheet: C1, C6, D1, J1, Q1, R1
